Commit message: more cleanup and name change

File: src/description/padih_bot.urdf.xacro (robot description, xacro)
@@ -1,4 +1,4 @@
 <?xml version="1.0"?>
-<robot name="agri_bot" xmlns:xacro="http://ros.org/wiki/xacro">
+<robot name="padih_bot" xmlns:xacro="http://ros.org/wiki/xacro">
     <xacro:property name="M_PI" value="3.1415926535897931"/>
     <xacro:arg name="namespace" default=" "/>
@@ -8,11 +8,9 @@
     <xacro:arg name="ros_domain_id" default=" "/>
     <xacro:property name="robot_id" value="$(arg ros_domain_id)"/>
-    <xacro:include filename="agri_bot_colors.xacro"/>
-    <xacro:include filename="agri_bot_inertias.xacro"/>
-    <xacro:include filename="agri_bot_core.xacro"/>
+    <xacro:include filename="padih_bot_colors.xacro"/>
+    <xacro:include filename="padih_bot_inertias.xacro"/>
+    <xacro:include filename="padih_bot_core.xacro"/>
     <xacro:include filename="gps.xacro"/>
     <xacro:include filename="OS1-32.xacro"/>
-    <!--        <xacro:include filename="camera.xacro" />-->
-    <!-- <xacro:include filename="gazebo_diff_drive_control.xacro" /> -->
     <xacro:include filename="agribot_diffdrive_control.xacro"/>
 </robot>

File: src/description/padih_bot_core.xacro (robot description, xacro)
@@ -12,5 +12,5 @@
             <origin xyz="0 0 0" rpy="0 0 0"/>
             <geometry>
-                <mesh filename="package://agri_bot/src/meshes/base_link.STL"/>
+                <mesh filename="package://padih_bot/src/meshes/base_link.STL"/>
             </geometry>
             <material name="green"/>
@@ -19,5 +19,5 @@
             <origin xyz="0 0 0" rpy="0 0 0"/>
             <geometry>
-                <mesh filename="package://agri_bot/src/meshes/base_link.STL"/>
+                <mesh filename="package://padih_bot/src/meshes/base_link.STL"/>
             </geometry>
         </collision>
@@ -42,5 +42,5 @@
             <origin xyz="0 0 0" rpy="0 0 0"/>
             <geometry>
-                <mesh filename="package://agri_bot/src/meshes/turret_link.STL"/>
+                <mesh filename="package://padih_bot/src/meshes/turret_link.STL"/>
             </geometry>
             <material name="yellow"/>
@@ -49,5 +49,5 @@
             <origin xyz="0 0 0" rpy="0 0 0"/>
             <geometry>
-                <mesh filename="package://agri_bot/src/meshes/turret_link.STL"/>
+                <mesh filename="package://padih_bot/src/meshes/turret_link.STL"/>
             </geometry>
         </collision>
@@ -88,5 +88,5 @@
             <origin xyz="0 0 0" rpy="0 0 0"/>
             <geometry>
-                <mesh filename="package://agri_bot/src/meshes/lidar-link.STL"/>
+                <mesh filename="package://padih_bot/src/meshes/lidar-link.STL"/>
             </geometry>
             <material name="">
@@ -97,5 +97,5 @@
             <origin xyz="0 0 0" rpy="0 0 0"/>
             <geometry>
-                <mesh filename="package://agri_bot/src/meshes/lidar-link.STL"/>
+                <mesh filename="package://padih_bot/src/meshes/lidar-link.STL"/>
             </geometry>
         </collision>
@@ -119,5 +119,5 @@
             <origin xyz="0 0 0" rpy="0 0 0"/>
             <geometry>
-                <mesh filename="package://agri_bot/src/meshes/right_wheel_link.STL"/>
+                <mesh filename="package://padih_bot/src/meshes/right_wheel_link.STL"/>
             </geometry>
             <material name="blue"/>
@@ -126,5 +126,5 @@
             <origin xyz="0 0 0" rpy="0 0 0"/>
             <geometry>
-                <mesh filename="package://agri_bot/src/meshes/right_wheel_link.STL"/>
+                <mesh filename="package://padih_bot/src/meshes/right_wheel_link.STL"/>
             </geometry>
         </collision>
@@ -157,5 +157,5 @@
             <origin xyz="0 0 0" rpy="0 0 0"/>
             <geometry>
-                <mesh filename="package://agri_bot/src/meshes/left_wheel_link.STL"/>
+                <mesh filename="package://padih_bot/src/meshes/left_wheel_link.STL"/>
             </geometry>
             <material name="blue"/>
@@ -164,5 +164,5 @@
             <origin xyz="0 0 0" rpy="0 0 0"/>
             <geometry>
-                <mesh filename="package://agri_bot/src/meshes/left_wheel_link.STL"/>
+                <mesh filename="package://padih_bot/src/meshes/left_wheel_link.STL"/>
             </geometry>
         </collision>
@@ -195,5 +195,5 @@
             <origin xyz="0 0 0" rpy="0 0 0"/>
             <geometry>
-                <mesh filename="package://agri_bot/src/meshes/caster_wheel_link.STL"/>
+                <mesh filename="package://padih_bot/src/meshes/caster_wheel_link.STL"/>
             </geometry>
             <material name="cyan"/>
@@ -202,5 +202,5 @@
             <origin xyz="0 0 0" rpy="0 0 0"/>
             <geometry>
-                <mesh filename="package://agri_bot/src/meshes/caster_wheel_link.STL"/>
+                <mesh filename="package://padih_bot/src/meshes/caster_wheel_link.STL"/>
             </geometry>
         </collision>

File: src/description/padih_bot_diffdrive_control.xacro (robot description, xacro)
@@ -53,5 +53,5 @@
         <gazebo>
             <plugin name="gazebo_ros2_control" filename="libgazebo_ros2_control.so">
-                <parameters>$(find agri_bot)/config/diffdrive_controllers.yaml</parameters>
+                <parameters>$(find padih_bot)/config/diffdrive_controllers.yaml</parameters>
                 <ros>
                     <remapping>/diffbot_base_controller/odom:=/controller/odometry</remapping>
